File: Production/MicroMod_SAMD51-Panel.brd (EAGLE design)
At the start: 199.6 x 83.1 mm, 550 parts, among them J1 MICROMOD-2222, J10 MICROMOD-2222, J11 MICROMOD-2222, J12 MICROMOD-2222, J13 MICROMOD-2222, J14 MICROMOD-2222, J15 MICROMOD-2222, J16 MICROMOD-2222, J2 MICROMOD-2222, J3 MICROMOD-2222, J4 MICROMOD-2222, J5 MICROMOD-2222, J6 MICROMOD-2222, J7 MICROMOD-2222, J8 MICROMOD-2222, J9 MICROMOD-2222, U1 W25QXX128MBIT-6X5-NO_CENTER, U10 ATSAMD51J20A-A, U11 W25QXX128MBIT-6X5-NO_CENTER, U12 ATSAMD51J20A-A, U13 W25QXX128MBIT-6X5-NO_CENTER, U14 ATSAMD51J20A-A, U15 W25QXX128MBIT-6X5-NO_CENTER, U16 ATSAMD51J20A-A, U17 W25QXX128MBIT-6X5-NO_CENTER, U18 ATSAMD51J20A-A, U19 W25QXX128MBIT-6X5-NO_CENTER, U2 ATSAMD51J20A-A, U20 ATSAMD51J20A-A, U21 W25QXX128MBIT-6X5-NO_CENTER, U22 ATSAMD51J20A-A, U23 W25QXX128MBIT-6X5-NO_CENTER, U24 ATSAMD51J20A-A, U25 W25QXX128MBIT-6X5-NO_CENTER, U26 ATSAMD51J20A-A, U27 W25QXX128MBIT-6X5-NO_CENTER, U28 ATSAMD51J20A-A, U29 W25QXX128MBIT-6X5-NO_CENTER, U3 W25QXX128MBIT-6X5-NO_CENTER, U30 ATSAMD51J20A-A, U31 W25QXX128MBIT-6X5-NO_CENTER, U32 ATSAMD51J20A-A, U4 ATSAMD51J20A-A, U5 W25QXX128MBIT-6X5-NO_CENTER, U6 ATSAMD51J20A-A, U7 W25QXX128MBIT-6X5-NO_CENTER, U8 ATSAMD51J20A-A, U9 W25QXX128MBIT-6X5-NO_CENTER, Y1 32.768kHz, Y10 32.768kHz, Y11 32.768kHz, Y12 32.768kHz, Y13 32.768kHz, Y14 32.768kHz, Y15 32.768kHz, Y16 32.768kHz, Y2 32.768kHz, Y3 32.768kHz, Y4 32.768kHz, Y5 32.768kHz, Y6 32.768kHz, Y7 32.768kHz, Y8 32.768kHz, Y9 32.768kHz

Commit message: v12 panel
Connections:
- net !CS: now also J2.55; no longer J2.70
- net !CS1: now also J1.55; no longer J1.70
- net !CS10: now also J11.55; no longer J11.70
- net !CS11: now also J12.55; no longer J12.70
- net !CS12: now also J13.55; no longer J13.70
- net !CS13: now also J14.55; no longer J14.70
- net !CS14: now also J15.55; no longer J15.70
- net !CS15: now also J16.55; no longer J16.70
- net !CS2: now also J3.55; no longer J3.70
- net !CS3: now also J4.55; no longer J4.70
- net !CS4: now also J5.55; no longer J5.70
- net !CS5: now also J6.55; no longer J6.70
- net !CS6: now also J7.55; no longer J7.70
- net !CS7: now also J8.55; no longer J8.70
- net !CS8: now also J9.55; no longer J9.70
- net !CS9: now also J10.55; no longer J10.70
- net CIPO: now also J2.61; no longer J2.64
- net CIPO10: now also J6.61; no longer J6.64
- net CIPO12: now also J7.61; no longer J7.64
- net CIPO14: now also J8.61; no longer J8.64
- net CIPO16: now also J9.61; no longer J9.64
- net CIPO18: now also J10.61; no longer J10.64
- net CIPO2: now also J1.61; no longer J1.64
- net CIPO20: now also J11.61; no longer J11.64
- net CIPO22: now also J12.61; no longer J12.64
- net CIPO24: now also J13.61; no longer J13.64
- net CIPO26: now also J14.61; no longer J14.64
- net CIPO28: now also J15.61; no longer J15.64
- net CIPO30: now also J16.61; no longer J16.64
- net CIPO4: now also J3.61; no longer J3.64
- net CIPO6: now also J4.61; no longer J4.64
- net CIPO8: now also J5.61; no longer J5.64
- net COPI: now also J2.59; no longer J2.62
- net COPI10: now also J6.59; no longer J6.62
- net COPI12: now also J7.59; no longer J7.62
- net COPI14: now also J8.59; no longer J8.62
- net COPI16: now also J9.59; no longer J9.62
- net COPI18: now also J10.59; no longer J10.62
- net COPI2: now also J1.59; no longer J1.62
- net COPI20: now also J11.59; no longer J11.62
- net COPI22: now also J12.59; no longer J12.62
- net COPI24: now also J13.59; no longer J13.62
- net COPI26: now also J14.59; no longer J14.62
- net COPI28: now also J15.59; no longer J15.62
- net COPI30: now also J16.59; no longer J16.62
- net COPI4: now also J3.59; no longer J3.62
- net COPI6: now also J4.59; no longer J4.62
- net COPI8: now also J5.59; no longer J5.62
- net SCLK: now also J2.57; no longer J2.60
- net SCLK10: now also J6.57; no longer J6.60
- net SCLK12: now also J7.57; no longer J7.60
- net SCLK14: now also J8.57; no longer J8.60
- net SCLK16: now also J9.57; no longer J9.60
- net SCLK18: now also J10.57; no longer J10.60
- net SCLK2: now also J1.57; no longer J1.60
- net SCLK20: now also J11.57; no longer J11.60
- net SCLK22: now also J12.57; no longer J12.60
- net SCLK24: now also J13.57; no longer J13.60
- net SCLK26: now also J14.57; no longer J14.60
- net SCLK28: now also J15.57; no longer J15.60
- net SCLK30: now also J16.57; no longer J16.60
- net SCLK4: now also J3.57; no longer J3.60
- net SCLK6: now also J4.57; no longer J4.60
- net SCLK8: now also J5.57; no longer J5.60
Routing:
- net !CS7: track 8.78 -> 7.74 mm
- net !CS6: track 8.78 -> 7.74 mm
- net !CS5: track 8.78 -> 7.74 mm
- net !CS13: track 8.78 -> 7.74 mm
- net !CS12: track 8.78 -> 7.74 mm
- net !CS11: track 8.78 -> 7.74 mm
- net !CS15: track 8.78 -> 7.74 mm
- net !CS14: track 8.78 -> 7.74 mm
- net !CS10: track 8.78 -> 7.74 mm
- net !CS2: track 8.78 -> 7.74 mm
- net !CS: track 8.78 -> 7.74 mm
- net !CS1: track 8.78 -> 7.74 mm
- net !CS8: track 8.78 -> 7.74 mm
- net !CS9: track 8.78 -> 7.74 mm
- net !CS4: track 8.78 -> 7.74 mm
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Other:
- board text added: "v12"
- board text removed: "v11"

Commit message: v12 panel, take 2
Routing:
- net !CS9: vias 1 -> 0
- net !CS8: vias 1 -> 0
- net !CS7: vias 1 -> 0
- net !CS6: vias 1 -> 0
- net !CS5: vias 1 -> 0
- net !CS4: vias 1 -> 0
- net !CS3: vias 1 -> 0
- net !CS2: vias 1 -> 0
- net !CS15: vias 1 -> 0
- net !CS14: vias 1 -> 0
- net !CS13: vias 1 -> 0
- net !CS12: vias 1 -> 0
- net !CS11: vias 1 -> 0
- net !CS10: vias 1 -> 0
- net !CS1: vias 1 -> 0
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Changed lines of the file:
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@@
 </signal>
 <signal name="!CS">
-<via x="5.3278" y="7.1834" extent="1-16" drill="0.2"/>
 <contactref element="U2" pad="16"/>
 <wire x1="5.3478" y1="8.1" x2="5.3478" y2="7.2034" width="0.1016" layer="1"/>
@@
 </signal>
 <signal name="!CS1">
-<via x="27.834740625" y="7.1834" extent="1-16" drill="0.2"/>
 <contactref element="U4" pad="16"/>
 <wire x1="27.854740625" y1="8.1" x2="27.854740625" y2="7.2034" width="0.1016" layer="1"/>
@@
 </signal>
 <signal name="!CS2">
-<via x="50.34421875" y="7.1834" extent="1-16" drill="0.2"/>
 <contactref element="U6" pad="16"/>
 <wire x1="50.36421875" y1="8.1" x2="50.36421875" y2="7.2034" width="0.1016" layer="1"/>
@@
 </signal>
 <signal name="!CS3">
-<via x="72.851159375" y="7.1834" extent="1-16" drill="0.2"/>
 <contactref element="U8" pad="16"/>
 <wire x1="72.871159375" y1="8.1" x2="72.871159375" y2="7.2034" width="0.1016" layer="1"/>
@@
 </signal>
 <signal name="!CS4">
-<via x="95.360640625" y="7.1834" extent="1-16" drill="0.2"/>
 <contactref element="U10" pad="16"/>
 <wire x1="95.380640625" y1="8.1" x2="95.380640625" y2="7.2034" width="0.1016" layer="1"/>
@@
 </signal>
 <signal name="!CS5">
-<via x="117.86758125" y="7.1834" extent="1-16" drill="0.2"/>
 <contactref element="U12" pad="16"/>
 <wire x1="117.88758125" y1="8.1" x2="117.88758125" y2="7.2034" width="0.1016" layer="1"/>
@@
 </signal>
 <signal name="!CS6">
-<via x="140.377059375" y="7.1834" extent="1-16" drill="0.2"/>
 <contactref element="U14" pad="16"/>
 <wire x1="140.397059375" y1="8.1" x2="140.397059375" y2="7.2034" width="0.1016" layer="1"/>
@@
 </signal>
 <signal name="!CS7">
-<via x="162.884" y="7.1834" extent="1-16" drill="0.2"/>
 <contactref element="U16" pad="16"/>
 <wire x1="162.904" y1="8.1" x2="162.904" y2="7.2034" width="0.1016" layer="1"/>
@@
 </signal>
 <signal name="!CS8">
-<via x="16.671140625" y="62.6666" extent="1-16" drill="0.2"/>
 <contactref element="U18" pad="16"/>
 <wire x1="16.651140625" y1="61.75" x2="16.651140625" y2="62.6466" width="0.1016" layer="1"/>
@@
 </signal>
 <signal name="!CS9">
-<via x="39.18061875" y="62.6666" extent="1-16" drill="0.2"/>
 <contactref element="U20" pad="16"/>
 <wire x1="39.16061875" y1="61.75" x2="39.16061875" y2="62.6466" width="0.1016" layer="1"/>
@@
 </signal>
 <signal name="!CS10">
-<via x="61.687559375" y="62.6666" extent="1-16" drill="0.2"/>
 <contactref element="U22" pad="16"/>
 <wire x1="61.667559375" y1="61.75" x2="61.667559375" y2="62.6466" width="0.1016" layer="1"/>
@@
 </signal>
 <signal name="!CS11">
-<via x="84.197040625" y="62.6666" extent="1-16" drill="0.2"/>
 <contactref element="U24" pad="16"/>
 <wire x1="84.177040625" y1="61.75" x2="84.177040625" y2="62.6466" width="0.1016" layer="1"/>
@@
 </signal>
 <signal name="!CS12">
-<via x="106.70398125" y="62.6666" extent="1-16" drill="0.2"/>
 <contactref element="U26" pad="16"/>
 <wire x1="106.68398125" y1="61.75" x2="106.68398125" y2="62.6466" width="0.1016" layer="1"/>
@@
 </signal>
 <signal name="!CS13">
-<via x="129.213459375" y="62.6666" extent="1-16" drill="0.2"/>
 <contactref element="U28" pad="16"/>
 <wire x1="129.193459375" y1="61.75" x2="129.193459375" y2="62.6466" width="0.1016" layer="1"/>
@@
 </signal>
 <signal name="!CS14">
-<via x="151.7204" y="62.6666" extent="1-16" drill="0.2"/>
 <contactref element="U30" pad="16"/>
 <wire x1="151.7004" y1="61.75" x2="151.7004" y2="62.6466" width="0.1016" layer="1"/>
@@
 </signal>
 <signal name="!CS15">
-<via x="174.227340625" y="62.6666" extent="1-16" drill="0.2"/>
 <contactref element="U32" pad="16"/>
 <wire x1="174.207340625" y1="61.75" x2="174.207340625" y2="62.6466" width="0.1016" layer="1"/>

Commit message: Panel update
Parts:
- moved E$5 0.51 mm to (-2.62, 6.35)
- moved E$6 0.51 mm to (-2.62, 6.35)
Connections:
- net CAN_RXI11 renamed D81
- net CAN_RXI12 renamed D88
- net CAN_RXI13 renamed D95
- net CAN_RXI14 renamed D102
- net CAN_RXI15 renamed D109
- net CAN_TXO11 renamed D80
- net CAN_TXO12 renamed D87
- net CAN_TXO13 renamed D94
- net CAN_TXO14 renamed D101
- net CAN_TXO15 renamed D108
- net D+/USB_HOST_D+ renamed D+/USBHOST_D+
- net D+/USB_HOST_D+1 renamed D+/USBHOST_D+1
- net D+/USB_HOST_D+10 renamed D+/USBHOST_D+10
- net D+/USB_HOST_D+11 renamed D+/USBHOST_D+11
- net D+/USB_HOST_D+12 renamed D+/USBHOST_D+12
- net D+/USB_HOST_D+13 renamed D+/USBHOST_D+13
- net D+/USB_HOST_D+14 renamed D+/USBHOST_D+14
- net D+/USB_HOST_D+15 renamed D+/USBHOST_D+15
- net D+/USB_HOST_D+2 renamed D+/USBHOST_D+2
- net D+/USB_HOST_D+3 renamed D+/USBHOST_D+3
- net D+/USB_HOST_D+4 renamed D+/USBHOST_D+4
- net D+/USB_HOST_D+5 renamed D+/USBHOST_D+5
- net D+/USB_HOST_D+6 renamed D+/USBHOST_D+6
- net D+/USB_HOST_D+7 renamed D+/USBHOST_D+7
- net D+/USB_HOST_D+8 renamed D+/USBHOST_D+8
- net D+/USB_HOST_D+9 renamed D+/USBHOST_D+9
- net SCLK renamed SCK
- net SCLK1 renamed SCK1
- net SCLK10 renamed SCK10
- net SCLK11 renamed SCK11
- net SCLK12 renamed SCK12
- net SCLK13 renamed SCK13
- net SCLK14 renamed SCK14
- net SCLK15 renamed SCK15
- net SCLK16 renamed SCK16
- net SCLK17 renamed SCK17
- net SCLK18 renamed SCK18
- net SCLK19 renamed SCK19
- net SCLK2 renamed SCK2
- net SCLK20 renamed SCK20
- net SCLK21 renamed SCK21
- net SCLK22 renamed SCK22
- net SCLK23 renamed SCK23
- net SCLK24 renamed SCK24
- net SCLK25 renamed SCK25
- net SCLK26 renamed SCK26
- net SCLK27 renamed SCK27
- net SCLK28 renamed SCK28
- net SCLK29 renamed SCK29
- net SCLK3 renamed SCK3
- net SCLK30 renamed SCK30
- net SCLK31 renamed SCK31
- net SCLK4 renamed SCK4
- net SCLK5 renamed SCK5
- net SCLK6 renamed SCK6
- net SCLK7 renamed SCK7
- net SCLK8 renamed SCK8
- net SCLK9 renamed SCK9
- removed net CAN_RXI: J2.41, U2.28
- removed net CAN_RXI1: J1.41, U4.28
- removed net CAN_RXI10: J11.41, U22.28
- removed net CAN_RXI2: J3.41, U6.28
- removed net CAN_RXI3: J4.41, U8.28
- removed net CAN_RXI4: J5.41, U10.28
- removed net CAN_RXI5: J6.41, U12.28
- removed net CAN_RXI6: J7.41, U14.28
- removed net CAN_RXI7: J8.41, U16.28
- removed net CAN_RXI8: J9.41, U18.28
- removed net CAN_RXI9: J10.41, U20.28
- removed net CAN_TXO: J2.43, U2.27
- removed net CAN_TXO1: J1.43, U4.27
- removed net CAN_TXO10: J11.43, U22.27
- removed net CAN_TXO2: J3.43, U6.27
- removed net CAN_TXO3: J4.43, U8.27
- removed net CAN_TXO4: J5.43, U10.27
- removed net CAN_TXO5: J6.43, U12.27
- removed net CAN_TXO6: J7.43, U14.27
- removed net CAN_TXO7: J8.43, U16.27
- removed net CAN_TXO8: J9.43, U18.27
- removed net CAN_TXO9: J10.43, U20.27
- new net D100: J15.18, U30.6
- new net D103: J15.67, U30.31
- new net D104: J15.65, U30.32
- new net D105: R62.2, U32.44
- new net D106: J16.10, U32.5
- new net D107: J16.18, U32.6
- new net D110: J16.67, U32.31
- new net D111: J16.65, U32.32
- new net D82: J12.67, U24.31
- new net D83: J12.65, U24.32
- new net D84: R50.2, U26.44
- new net D85: J13.10, U26.5
- new net D86: J13.18, U26.6
- new net D89: J13.67, U26.31
- new net D90: J13.65, U26.32
- new net D91: R54.2, U28.44
- new net D92: J14.10, U28.5
- new net D93: J14.18, U28.6
- new net D96: J14.67, U28.31
- new net D97: J14.65, U28.32
- new net D98: R58.2, U30.44
- new net D99: J15.10, U30.5
- net CIPO1: now also U1.2; no longer U1.5
- net CIPO11: now also U11.2; no longer U11.5
- net CIPO13: now also U13.2; no longer U13.5
- net CIPO15: now also U15.2; no longer U15.5
- net CIPO17: now also U17.2; no longer U17.5
- net CIPO19: now also U19.2; no longer U19.5
- net CIPO21: now also U21.2; no longer U21.5
- net CIPO23: now also U23.2; no longer U23.5
- net CIPO25: now also U25.2; no longer U25.5
- net CIPO27: now also U27.2; no longer U27.5
- net CIPO29: now also U29.2; no longer U29.5
- net CIPO3: now also U3.2; no longer U3.5
- net CIPO31: now also U31.2; no longer U31.5
- net CIPO5: now also U5.2; no longer U5.5
- net CIPO7: now also U7.2; no longer U7.5
- net CIPO9: now also U9.2; no longer U9.5
- net COPI1: now also U1.5; no longer U1.2
- net COPI11: now also U11.5; no longer U11.2
- net COPI13: now also U13.5; no longer U13.2
- net COPI15: now also U15.5; no longer U15.2
- net COPI17: now also U17.5; no longer U17.2
- net COPI19: now also U19.5; no longer U19.2
- net COPI21: now also U21.5; no longer U21.2
- net COPI23: now also U23.5; no longer U23.2
- net COPI25: now also U25.5; no longer U25.2
- net COPI27: now also U27.5; no longer U27.2
- net COPI29: now also U29.5; no longer U29.2
- net COPI3: now also U3.5; no longer U3.2
- net COPI31: now also U31.5; no longer U31.2
- net COPI5: now also U5.5; no longer U5.2
- net COPI7: now also U7.5; no longer U7.2
- net COPI9: now also U9.5; no longer U9.2
- net D12: now also J3.10, U6.5; no longer J3.67, U6.31
- net D14: now also J3.18, U6.6; no longer J3.65, U6.32
- net D15: now also J3.43, U6.27; no longer R14.2, U8.44
- net D16: now also J3.41, U6.28; no longer J4.10, U8.5
- net D17: now also J3.67, U6.31; no longer J4.18, U8.6
- net D18: now also J3.65, U6.32; no longer J4.67, U8.31
- net D19: now also R14.2, U8.44; no longer J4.65, U8.32
- net D20: now also J4.10, U8.5; no longer R18.2, U10.44
- net D21: now also J4.18, U8.6; no longer J5.10, U10.5
- net D22: now also J4.43, U8.27; no longer J5.18, U10.6
- net D23: now also J4.41, U8.28; no longer J5.67, U10.31
- net D24: now also J4.67, U8.31; no longer J5.65, U10.32
- net D25: now also J4.65, U8.32; no longer R22.2, U12.44
- net D26: now also R18.2, U10.44; no longer J6.10, U12.5
- net D27: now also J5.10, U10.5; no longer J6.18, U12.6
- net D28: now also J5.18, U10.6; no longer J6.67, U12.31
- net D29: now also J5.43, U10.27; no longer J6.65, U12.32
- net D30: now also J5.41, U10.28; no longer R26.2, U14.44
- net D31: now also J5.67, U10.31; no longer J7.10, U14.5
- net D32: now also J5.65, U10.32; no longer J7.18, U14.6
- net D33: now also R22.2, U12.44; no longer J7.67, U14.31
- net D34: now also J6.10, U12.5; no longer J7.65, U14.32
- net D35: now also J6.18, U12.6; no longer R30.2, U16.44
- net D36: now also J6.43, U12.27; no longer J8.10, U16.5
- net D37: now also J6.41, U12.28; no longer J8.18, U16.6
- net D38: now also J2.43, U2.27; no longer J8.67, U16.31
- net D39: now also J2.41, U2.28; no longer J8.65, U16.32
- net D40: now also J6.67, U12.31; no longer R34.2, U18.44
- net D41: now also J6.65, U12.32; no longer J9.10, U18.5
- net D42: now also R26.2, U14.44; no longer J9.18, U18.6
- net D43: now also J7.10, U14.5; no longer J9.67, U18.31
- net D44: now also J7.18, U14.6; no longer J9.65, U18.32
- net D45: now also J7.43, U14.27; no longer R38.2, U20.44
- net D46: now also J7.41, U14.28; no longer J10.10, U20.5
- net D47: now also J7.67, U14.31; no longer J10.18, U20.6
- net D48: now also J7.65, U14.32; no longer J10.67, U20.31
- net D49: now also R30.2, U16.44; no longer J10.65, U20.32
- net D5: now also J1.43, U4.27; no longer J1.67, U4.31
- net D50: now also J8.10, U16.5; no longer R42.2, U22.44
- net D51: now also J8.18, U16.6; no longer J11.10, U22.5
- net D52: now also J8.43, U16.27; no longer J11.18, U22.6
- net D53: now also J8.41, U16.28; no longer J11.67, U22.31
- net D54: now also J8.67, U16.31; no longer J11.65, U22.32
- net D55: now also J8.65, U16.32; no longer R46.2, U24.44
- net D56: now also R34.2, U18.44; no longer J12.10, U24.5
- net D57: now also J9.10, U18.5; no longer J12.18, U24.6
- net D58: now also J9.18, U18.6; no longer J12.67, U24.31
- net D59: now also J9.43, U18.27; no longer J12.65, U24.32
- net D6: now also J1.41, U4.28; no longer J1.65, U4.32
- net D60: now also J9.41, U18.28; no longer R50.2, U26.44
- net D61: now also J9.67, U18.31; no longer J13.10, U26.5
- net D62: now also J9.65, U18.32; no longer J13.18, U26.6
- net D63: now also R38.2, U20.44; no longer J13.67, U26.31
- net D64: now also J10.10, U20.5; no longer J13.65, U26.32
- net D65: now also J10.18, U20.6; no longer R54.2, U28.44
- net D66: now also J10.43, U20.27; no longer J14.10, U28.5
- net D67: now also J10.41, U20.28; no longer J14.18, U28.6
- net D68: now also J10.67, U20.31; no longer J14.67, U28.31
- net D69: now also J10.65, U20.32; no longer J14.65, U28.32
- net D7: now also J1.67, U4.31; no longer R10.2, U6.44
- net D70: now also R42.2, U22.44; no longer R58.2, U30.44
- net D71: now also J11.10, U22.5; no longer J15.10, U30.5
- net D72: now also J11.18, U22.6; no longer J15.18, U30.6
- net D73: now also J11.43, U22.27; no longer J15.67, U30.31
- net D74: now also J11.41, U22.28; no longer J15.65, U30.32
- net D75: now also J11.67, U22.31; no longer R62.2, U32.44
- net D76: now also J11.65, U22.32; no longer J16.10, U32.5
- net D77: now also R46.2, U24.44; no longer J16.18, U32.6
- net D78: now also J12.10, U24.5; no longer J16.67, U32.31
- net D79: now also J12.18, U24.6; no longer J16.65, U32.32
- net D8: now also J1.65, U4.32; no longer J3.10, U6.5
- net D9: now also R10.2, U6.44; no longer J3.18, U6.6
Routing:
- net D91: track 0.00 -> 22.4 mm, vias 0 -> 2
- net D98: track 0.00 -> 22.4 mm, vias 0 -> 2
- net D105: track 0.00 -> 22.4 mm, vias 0 -> 2
- net D84: track 0.00 -> 22.4 mm, vias 0 -> 2
- net D99: track 0.00 -> 22.3 mm, vias 0 -> 2
- net D106: track 0.00 -> 22.3 mm, vias 0 -> 2
- net D92: track 0.00 -> 22.3 mm, vias 0 -> 2
- net D85: track 0.00 -> 22.3 mm, vias 0 -> 2
- net D93: track 0.00 -> 21.0 mm, vias 0 -> 2
- net D86: track 0.00 -> 21.0 mm, vias 0 -> 2
- net D107: track 0.00 -> 21.0 mm, vias 0 -> 2
- net D100: track 0.00 -> 21.0 mm, vias 0 -> 2
- net D89: track 0.00 -> 18.9 mm, vias 0 -> 3
- net D82: track 0.00 -> 18.9 mm, vias 0 -> 3
- net D96: track 0.00 -> 18.9 mm, vias 0 -> 3
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Other:
- board text added: "v13"
- board text removed: "v12"
